Commit message: updated rbkairos xacro file
updated rbkairos xacro file to include the tool

File: rbkairos_tc/rbkairos_common/rbkairos_description/robots/rbkairos.urdf.xacro (robot description, xacro)
@@ -16,4 +16,6 @@
 	<!-- Include UR-10 ARM -->
 	<xacro:include filename="$(find ur_description)/urdf/ur10.urdf.xacro" />
+	<!-- Include SPRAY TOOL -->
+	<xacro:include filename="$(find spray_tool_description)/urdf/spray_tool.xacro" />
     <!-- Arm Camera -->
     <xacro:include filename="$(find robotnik_sensors)/urdf/kinect.urdf.xacro" />
@@ -143,4 +145,8 @@
 			</joint>
 		</xacro:if>
+		<!-- SPRAY TOOL -->
+		<xacro:spray_tool prefix="$(arg prefix)spray_tool" parent="$(arg prefix)ur10_tool0">
+			<origin xyz="0.0 0.0 0.0" rpy="0 0 0"/>
+		</xacro:spray_tool>
 		<!-- Schunk WSG-50 -->
         <xacro:if value="$(arg has_gripper)">
